File: RP2040-mcu.kicad_sch (KiCad schematic)
At the start: 34 parts, among them J1 Conn_01x04, J2 Conn_01x05, J3 Conn_01x11, J4 Conn_01x11, J5 Conn_01x11, SW1 SW_Push, U1 W25Q128JVS, U2 RP2040, U3 XC6206PxxxMR-Regulator_Linear, Y1 Crystal_GND24_Small

Commit message: Assigned footprints
Macropad + RP2040
Parts:
- R2: footprint (none) -> Resistor_SMD:R_0402_1005Metric
- U2: footprint Sleep-Lib:RP2040-QFN-56 -> Sleep-footprints:RP2040-QFN-56
Changed lines of the file:
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@@
     (property "Reference" "U2" (id 0) (at 68.58 127 0))
     (property "Value" "RP2040" (id 1) (at 68.58 129.54 0))
-    (property "Footprint" "Sleep-Lib:RP2040-QFN-56" (id 2) (at 48.26 13.97 0)
+    (property "Footprint" "Sleep-footprints:RP2040-QFN-56" (id 2) (at 48.26 13.97 0)
       (effects (font (size 1.27 1.27)) (justify left bottom) hide)
     )
@@
       (effects (font (size 1.27 1.27)) (justify left))
     )
-    (property "Footprint" "" (id 2) (at 35.56 29.21 0)
-      (effects (font (size 1.27 1.27)) hide)
-    )
+    (property "Footprint" "Resistor_SMD:R_0402_1005Metric" (id 2) (at 35.56 29.21 0)
+      (effects (font (size 1.27 1.27)) hide)
+    )
