File: MacroPad.kicad_sch (KiCad schematic)
At the start: 54 parts, among them K1 Mod1, K10 8, K11 9, K12 SW_Push, K13 4, K14 5, K15 6, K16 SW_Push, K17 1, K18 2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

Commit message: Assigned footprints
Macropad + RP2040
Parts:
- F1, F2: footprint (none) -> Connector_PinHeader_2.54mm:PinHeader_1x04_P2.54mm_Vertical
- K10, K11, K12, K13, K14, K15, K16, K17, K18, K19, K20, K21, K22, K23, K24, K5, K6, K7, K8, K9, KO-1, KO-2, KO-3, KO-4: footprint (none) -> marbastlib-mx:SW_MX_HS_1u
Changed lines of the file:
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@@
       (effects (font (size 1.27 1.27)) hide)
     )
-    (property "Footprint" "" (id 2) (at 111.76 96.52 0)
+    (property "Footprint" "marbastlib-mx:SW_MX_HS_1u" (id 2) (at 111.76 96.52 0)
       (effects (font (size 1.27 1.27)) hide)
     )
@@
       (effects (font (size 1.27 1.27)) hide)
     )
-    (property "Footprint" "" (id 2) (at 140.97 148.59 0)
+    (property "Footprint" "marbastlib-mx:SW_MX_HS_1u" (id 2) (at 140.97 148.59 0)
       (effects (font (size 1.27 1.27)) hide)
     )
@@
       (effects (font (size 1.27 1.27)) hide)
     )
-    (property "Footprint" "" (id 2) (at 67.31 134.62 0)
+    (property "Footprint" "marbastlib-mx:SW_MX_HS_1u" (id 2) (at 67.31 134.62 0)
       (effects (font (size 1.27 1.27)) hide)
     )
@@
       (effects (font (size 1.27 1.27)) hide)
     )
-    (property "Footprint" "" (id 2) (at 96.52 82.55 0)
+    (property "Footprint" "marbastlib-mx:SW_MX_HS_1u" (id 2) (at 96.52 82.55 0)
       (effects (font (size 1.27 1.27)) hide)
     )
@@
       (effects (font (size 1.27 1.27)) hide)
     )
-    (property "Footprint" "" (id 2) (at 111.76 110.49 0)
+    (property "Footprint" "marbastlib-mx:SW_MX_HS_1u" (id 2) (at 111.76 110.49 0)
       (effects (font (size 1.27 1.27)) hide)
     )
@@
       (effects (font (size 1.27 1.27)) hide)
     )
-    (property "Footprint" "" (id 2) (at 67.31 120.65 0)
+    (property "Footprint" "marbastlib-mx:SW_MX_HS_1u" (id 2) (at 67.31 120.65 0)
       (effects (font (size 1.27 1.27)) hide)
     )
@@
       (effects (font (size 1.27 1.27)) hide)
     )
-    (property "Footprint" "" (id 2) (at 140.97 120.65 0)
+    (property "Footprint" "marbastlib-mx:SW_MX_HS_1u" (id 2) (at 140.97 120.65 0)
       (effects (font (size 1.27 1.27)) hide)
     )
@@
       (effects (font (size 1.27 1.27)) hide)
     )
-    (property "Footprint" "" (id 2) (at 111.76 82.55 0)
+    (property "Footprint" "marbastlib-mx:SW_MX_HS_1u" (id 2) (at 111.76 82.55 0)
       (effects (font (size 1.27 1.27)) hide)
     )
@@
       (effects (font (size 1.27 1.27)) hide)
     )
-    (property "Footprint" "" (id 2) (at 96.52 96.52 0)
+    (property "Footprint" "marbastlib-mx:SW_MX_HS_1u" (id 2) (at 96.52 96.52 0)
       (effects (font (size 1.27 1.27)) hide)
     )
@@
       (effects (font (size 1.27 1.27)) hide)
     )
-    (property "Footprint" "" (id 2) (at 127 138.43 0)
+    (property "Footprint" "marbastlib-mx:SW_MX_HS_1u" (id 2) (at 127 138.43 0)
       (effects (font (size 1.27 1.27)) hide)
     )
@@
       (effects (font (size 1.27 1.27)) hide)
     )
-    (property "Footprint" "" (id 2) (at 96.52 110.49 0)
+    (property "Footprint" "marbastlib-mx:SW_MX_HS_1u" (id 2) (at 96.52 110.49 0)
       (effects (font (size 1.27 1.27)) hide)
     )
@@
       (effects (font (size 1.27 1.27)) hide)
     )
-    (property "Footprint" "" (id 2) (at 111.76 124.46 0)
+    (property "Footprint" "marbastlib-mx:SW_MX_HS_1u" (id 2) (at 111.76 124.46 0)
       (effects (font (size 1.27 1.27)) hide)
     )
@@
       (effects (font (size 1.27 1.27)) hide)
     )
-    (property "Footprint" "" (id 2) (at 81.28 138.43 0)
+    (property "Footprint" "marbastlib-mx:SW_MX_HS_1u" (id 2) (at 81.28 138.43 0)
       (effects (font (size 1.27 1.27)) hide)
     )
@@
       (effects (font (size 1.27 1.27)) hide)
     )
-    (property "Footprint" "" (id 2) (at 127 124.46 0)
+    (property "Footprint" "marbastlib-mx:SW_MX_HS_1u" (id 2) (at 127 124.46 0)
       (effects (font (size 1.27 1.27)) hide)
     )
@@
       (effects (font (size 1.27 1.27)) hide)
     )
-    (property "Footprint" "" (id 2) (at 127 110.49 0)
+    (property "Footprint" "marbastlib-mx:SW_MX_HS_1u" (id 2) (at 127 110.49 0)
       (effects (font (size 1.27 1.27)) hide)
     )
@@
       (effects (font (size 1.27 1.27)) hide)
     )
-    (property "Footprint" "" (id 2) (at 81.28 82.55 0)
+    (property "Footprint" "marbastlib-mx:SW_MX_HS_1u" (id 2) (at 81.28 82.55 0)
       (effects (font (size 1.27 1.27)) hide)
     )
@@
       (effects (font (size 1.27 1.27)) hide)
     )
-    (property "Footprint" "" (id 2) (at 96.52 124.46 0)
+    (property "Footprint" "marbastlib-mx:SW_MX_HS_1u" (id 2) (at 96.52 124.46 0)
       (effects (font (size 1.27 1.27)) hide)
     )
@@
     (property "Reference" "F2" (id 0) (at 103.505 24.13 0))
     (property "Value" "OLED2" (id 1) (at 103.505 26.67 0))
-    (property "Footprint" "" (id 2) (at 102.87 31.75 0)
+    (property "Footprint" "Connector_PinHeader_2.54mm:PinHeader_1x04_P2.54mm_Vertical" (id 2) (at 102.87 31.75 0)
       (effects (font (size 1.27 1.27)) hide)
     )
@@
     (property "Reference" "F1" (id 0) (at 81.915 24.13 0))
     (property "Value" "OLED1" (id 1) (at 81.915 26.67 0))
-    (property "Footprint" "" (id 2) (at 81.28 31.75 0)
+    (property "Footprint" "Connector_PinHeader_2.54mm:PinHeader_1x04_P2.54mm_Vertical" (id 2) (at 81.28 31.75 0)
       (effects (font (size 1.27 1.27)) hide)
     )
@@
       (effects (font (size 1.27 1.27)) hide)
     )
-    (property "Footprint" "" (id 2) (at 96.52 138.43 0)
+    (property "Footprint" "marbastlib-mx:SW_MX_HS_1u" (id 2) (at 96.52 138.43 0)
       (effects (font (size 1.27 1.27)) hide)
     )
@@
       (effects (font (size 1.27 1.27)) hide)
     )
-    (property "Footprint" "" (id 2) (at 81.28 96.52 0)
+    (property "Footprint" "marbastlib-mx:SW_MX_HS_1u" (id 2) (at 81.28 96.52 0)
       (effects (font (size 1.27 1.27)) hide)
     )
@@
       (effects (font (size 1.27 1.27)) hide)
     )
-    (property "Footprint" "" (id 2) (at 81.28 110.49 0)
+    (property "Footprint" "marbastlib-mx:SW_MX_HS_1u" (id 2) (at 81.28 110.49 0)
       (effects (font (size 1.27 1.27)) hide)
     )
@@
       (effects (font (size 1.27 1.27)) hide)
     )
-    (property "Footprint" "" (id 2) (at 127 82.55 0)
+    (property "Footprint" "marbastlib-mx:SW_MX_HS_1u" (id 2) (at 127 82.55 0)
       (effects (font (size 1.27 1.27)) hide)
     )
@@
       (effects (font (size 1.27 1.27)) hide)
     )
-    (property "Footprint" "" (id 2) (at 111.76 138.43 0)
+    (property "Footprint" "marbastlib-mx:SW_MX_HS_1u" (id 2) (at 111.76 138.43 0)
       (effects (font (size 1.27 1.27)) hide)
     )
@@
       (effects (font (size 1.27 1.27)) hide)
     )
-    (property "Footprint" "" (id 2) (at 81.28 124.46 0)
+    (property "Footprint" "marbastlib-mx:SW_MX_HS_1u" (id 2) (at 81.28 124.46 0)
       (effects (font (size 1.27 1.27)) hide)
     )
@@
       (effects (font (size 1.27 1.27)) hide)
     )
-    (property "Footprint" "" (id 2) (at 127 96.52 0)
-      (effects (font (size 1.27 1.27)) hide)
-    )
+    (property "Footprint" "marbastlib-mx:SW_MX_HS_1u" (id 2) (at 127 96.52 0)
+      (effects (font (size 1.27 1.27)) hide)
+    )

Commit message: Modified enc footprint
Parts:
- K1, K2, K3, K4: footprint marbastlib-mx:SW_MX_HS_1u_Enc -> Switch_Keyboard_Hotswap_Kailh:SW_Hotswap_Kailh_MX_plated_1.00u_Enc
- K10, K11, K12, K13, K14, K15, K16, K17, K18, K19, K20, K21, K22, K23, K24, K5, K6, K7, K8, K9, KO-1, KO-2, KO-3, KO-4: footprint marbastlib-mx:SW_MX_HS_1u -> Switch_Keyboard_Hotswap_Kailh:SW_Hotswap_Kailh_MX_plated_1.00u
Changed lines of the file:
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@@
     (property "Reference" "K2" (id 0) (at 87.63 49.53 0))
     (property "Value" "Mod2" (id 1) (at 87.63 52.07 0))
-    (property "Footprint" "marbastlib-mx:SW_MX_HS_1u_Enc" (id 2) (at 91.44 63.754 0)
+    (property "Footprint" "Switch_Keyboard_Hotswap_Kailh:SW_Hotswap_Kailh_MX_plated_1.00u_Enc" (id 2) (at 91.44 63.754 0)
       (effects (font (size 1.27 1.27)) hide)
     )
@@
       (effects (font (size 1.27 1.27)) hide)
     )
-    (property "Footprint" "marbastlib-mx:SW_MX_HS_1u" (id 2) (at 111.76 96.52 0)
+    (property "Footprint" "Switch_Keyboard_Hotswap_Kailh:SW_Hotswap_Kailh_MX_plated_1.00u" (id 2) (at 111.76 96.52 0)
       (effects (font (size 1.27 1.27)) hide)
     )
@@
       (effects (font (size 1.27 1.27)) hide)
     )
-    (property "Footprint" "marbastlib-mx:SW_MX_HS_1u" (id 2) (at 140.97 148.59 0)
+    (property "Footprint" "Switch_Keyboard_Hotswap_Kailh:SW_Hotswap_Kailh_MX_plated_1.00u" (id 2) (at 140.97 148.59 0)
       (effects (font (size 1.27 1.27)) hide)
     )
@@
       (effects (font (size 1.27 1.27)) hide)
     )
-    (property "Footprint" "marbastlib-mx:SW_MX_HS_1u" (id 2) (at 67.31 134.62 0)
+    (property "Footprint" "Switch_Keyboard_Hotswap_Kailh:SW_Hotswap_Kailh_MX_plated_1.00u" (id 2) (at 67.31 134.62 0)
       (effects (font (size 1.27 1.27)) hide)
     )
@@
       (effects (font (size 1.27 1.27)) hide)
     )
-    (property "Footprint" "marbastlib-mx:SW_MX_HS_1u" (id 2) (at 96.52 82.55 0)
+    (property "Footprint" "Switch_Keyboard_Hotswap_Kailh:SW_Hotswap_Kailh_MX_plated_1.00u" (id 2) (at 96.52 82.55 0)
       (effects (font (size 1.27 1.27)) hide)
     )
@@
       (effects (font (size 1.27 1.27)) hide)
     )
-    (property "Footprint" "marbastlib-mx:SW_MX_HS_1u" (id 2) (at 111.76 110.49 0)
+    (property "Footprint" "Switch_Keyboard_Hotswap_Kailh:SW_Hotswap_Kailh_MX_plated_1.00u" (id 2) (at 111.76 110.49 0)
       (effects (font (size 1.27 1.27)) hide)
     )
@@
       (effects (font (size 1.27 1.27)) hide)
     )
-    (property "Footprint" "marbastlib-mx:SW_MX_HS_1u" (id 2) (at 67.31 120.65 0)
+    (property "Footprint" "Switch_Keyboard_Hotswap_Kailh:SW_Hotswap_Kailh_MX_plated_1.00u" (id 2) (at 67.31 120.65 0)
       (effects (font (size 1.27 1.27)) hide)
     )
@@
       (effects (font (size 1.27 1.27)) hide)
     )
-    (property "Footprint" "marbastlib-mx:SW_MX_HS_1u" (id 2) (at 140.97 120.65 0)
+    (property "Footprint" "Switch_Keyboard_Hotswap_Kailh:SW_Hotswap_Kailh_MX_plated_1.00u" (id 2) (at 140.97 120.65 0)
       (effects (font (size 1.27 1.27)) hide)
     )
@@
       (effects (font (size 1.27 1.27)) hide)
     )
-    (property "Footprint" "marbastlib-mx:SW_MX_HS_1u" (id 2) (at 111.76 82.55 0)
+    (property "Footprint" "Switch_Keyboard_Hotswap_Kailh:SW_Hotswap_Kailh_MX_plated_1.00u" (id 2) (at 111.76 82.55 0)
       (effects (font (size 1.27 1.27)) hide)
     )
@@
       (effects (font (size 1.27 1.27)) hide)
     )
-    (property "Footprint" "marbastlib-mx:SW_MX_HS_1u" (id 2) (at 96.52 96.52 0)
+    (property "Footprint" "Switch_Keyboard_Hotswap_Kailh:SW_Hotswap_Kailh_MX_plated_1.00u" (id 2) (at 96.52 96.52 0)
       (effects (font (size 1.27 1.27)) hide)
     )
@@
       (effects (font (size 1.27 1.27)) hide)
     )
-    (property "Footprint" "marbastlib-mx:SW_MX_HS_1u" (id 2) (at 127 138.43 0)
+    (property "Footprint" "Switch_Keyboard_Hotswap_Kailh:SW_Hotswap_Kailh_MX_plated_1.00u" (id 2) (at 127 138.43 0)
       (effects (font (size 1.27 1.27)) hide)
     )
@@
       (effects (font (size 1.27 1.27)) hide)
     )
-    (property "Footprint" "marbastlib-mx:SW_MX_HS_1u" (id 2) (at 96.52 110.49 0)
+    (property "Footprint" "Switch_Keyboard_Hotswap_Kailh:SW_Hotswap_Kailh_MX_plated_1.00u" (id 2) (at 96.52 110.49 0)
       (effects (font (size 1.27 1.27)) hide)
     )
@@
     (property "Reference" "K4" (id 0) (at 143.51 49.53 0))
     (property "Value" "Mod4" (id 1) (at 143.51 52.07 0))
-    (property "Footprint" "marbastlib-mx:SW_MX_HS_1u_Enc" (id 2) (at 147.32 63.754 0)
+    (property "Footprint" "Switch_Keyboard_Hotswap_Kailh:SW_Hotswap_Kailh_MX_plated_1.00u_Enc" (id 2) (at 147.32 63.754 0)
       (effects (font (size 1.27 1.27)) hide)
     )
@@
       (effects (font (size 1.27 1.27)) hide)
     )
-    (property "Footprint" "marbastlib-mx:SW_MX_HS_1u" (id 2) (at 111.76 124.46 0)
+    (property "Footprint" "Switch_Keyboard_Hotswap_Kailh:SW_Hotswap_Kailh_MX_plated_1.00u" (id 2) (at 111.76 124.46 0)
       (effects (font (size 1.27 1.27)) hide)
     )
@@
     (property "Reference" "K1" (id 0) (at 59.69 49.53 0))
     (property "Value" "Mod1" (id 1) (at 59.69 52.07 0))
-    (property "Footprint" "marbastlib-mx:SW_MX_HS_1u_Enc" (id 2) (at 63.5 63.754 0)
+    (property "Footprint" "Switch_Keyboard_Hotswap_Kailh:SW_Hotswap_Kailh_MX_plated_1.00u_Enc" (id 2) (at 63.5 63.754 0)
       (effects (font (size 1.27 1.27)) hide)
     )
@@
       (effects (font (size 1.27 1.27)) hide)
     )
-    (property "Footprint" "marbastlib-mx:SW_MX_HS_1u" (id 2) (at 81.28 138.43 0)
+    (property "Footprint" "Switch_Keyboard_Hotswap_Kailh:SW_Hotswap_Kailh_MX_plated_1.00u" (id 2) (at 81.28 138.43 0)
       (effects (font (size 1.27 1.27)) hide)
     )
@@
       (effects (font (size 1.27 1.27)) hide)
     )
-    (property "Footprint" "marbastlib-mx:SW_MX_HS_1u" (id 2) (at 127 124.46 0)
+    (property "Footprint" "Switch_Keyboard_Hotswap_Kailh:SW_Hotswap_Kailh_MX_plated_1.00u" (id 2) (at 127 124.46 0)
       (effects (font (size 1.27 1.27)) hide)
     )
@@
       (effects (font (size 1.27 1.27)) hide)
     )
-    (property "Footprint" "marbastlib-mx:SW_MX_HS_1u" (id 2) (at 127 110.49 0)
+    (property "Footprint" "Switch_Keyboard_Hotswap_Kailh:SW_Hotswap_Kailh_MX_plated_1.00u" (id 2) (at 127 110.49 0)
       (effects (font (size 1.27 1.27)) hide)
     )
@@
       (effects (font (size 1.27 1.27)) hide)
     )
-    (property "Footprint" "marbastlib-mx:SW_MX_HS_1u" (id 2) (at 81.28 82.55 0)
+    (property "Footprint" "Switch_Keyboard_Hotswap_Kailh:SW_Hotswap_Kailh_MX_plated_1.00u" (id 2) (at 81.28 82.55 0)
       (effects (font (size 1.27 1.27)) hide)
     )
@@
       (effects (font (size 1.27 1.27)) hide)
     )
-    (property "Footprint" "marbastlib-mx:SW_MX_HS_1u" (id 2) (at 96.52 124.46 0)
+    (property "Footprint" "Switch_Keyboard_Hotswap_Kailh:SW_Hotswap_Kailh_MX_plated_1.00u" (id 2) (at 96.52 124.46 0)
       (effects (font (size 1.27 1.27)) hide)
     )
@@
       (effects (font (size 1.27 1.27)) hide)
     )
-    (property "Footprint" "marbastlib-mx:SW_MX_HS_1u" (id 2) (at 96.52 138.43 0)
+    (property "Footprint" "Switch_Keyboard_Hotswap_Kailh:SW_Hotswap_Kailh_MX_plated_1.00u" (id 2) (at 96.52 138.43 0)
       (effects (font (size 1.27 1.27)) hide)
     )
@@
       (effects (font (size 1.27 1.27)) hide)
     )
-    (property "Footprint" "marbastlib-mx:SW_MX_HS_1u" (id 2) (at 81.28 96.52 0)
+    (property "Footprint" "Switch_Keyboard_Hotswap_Kailh:SW_Hotswap_Kailh_MX_plated_1.00u" (id 2) (at 81.28 96.52 0)
       (effects (font (size 1.27 1.27)) hide)
     )
@@
       (effects (font (size 1.27 1.27)) hide)
     )
-    (property "Footprint" "marbastlib-mx:SW_MX_HS_1u" (id 2) (at 81.28 110.49 0)
+    (property "Footprint" "Switch_Keyboard_Hotswap_Kailh:SW_Hotswap_Kailh_MX_plated_1.00u" (id 2) (at 81.28 110.49 0)
       (effects (font (size 1.27 1.27)) hide)
     )
@@
     (property "Reference" "K3" (id 0) (at 115.57 49.53 0))
     (property "Value" "Mod3" (id 1) (at 115.57 52.07 0))
-    (property "Footprint" "marbastlib-mx:SW_MX_HS_1u_Enc" (id 2) (at 119.38 63.754 0)
+    (property "Footprint" "Switch_Keyboard_Hotswap_Kailh:SW_Hotswap_Kailh_MX_plated_1.00u_Enc" (id 2) (at 119.38 63.754 0)
       (effects (font (size 1.27 1.27)) hide)
     )
@@
       (effects (font (size 1.27 1.27)) hide)
     )
-    (property "Footprint" "marbastlib-mx:SW_MX_HS_1u" (id 2) (at 127 82.55 0)
+    (property "Footprint" "Switch_Keyboard_Hotswap_Kailh:SW_Hotswap_Kailh_MX_plated_1.00u" (id 2) (at 127 82.55 0)
       (effects (font (size 1.27 1.27)) hide)
     )
@@
       (effects (font (size 1.27 1.27)) hide)
     )
-    (property "Footprint" "marbastlib-mx:SW_MX_HS_1u" (id 2) (at 111.76 138.43 0)
+    (property "Footprint" "Switch_Keyboard_Hotswap_Kailh:SW_Hotswap_Kailh_MX_plated_1.00u" (id 2) (at 111.76 138.43 0)
       (effects (font (size 1.27 1.27)) hide)
     )
@@
       (effects (font (size 1.27 1.27)) hide)
     )
-    (property "Footprint" "marbastlib-mx:SW_MX_HS_1u" (id 2) (at 81.28 124.46 0)
+    (property "Footprint" "Switch_Keyboard_Hotswap_Kailh:SW_Hotswap_Kailh_MX_plated_1.00u" (id 2) (at 81.28 124.46 0)
       (effects (font (size 1.27 1.27)) hide)
     )
@@
       (effects (font (size 1.27 1.27)) hide)
     )
-    (property "Footprint" "marbastlib-mx:SW_MX_HS_1u" (id 2) (at 127 96.52 0)
-      (effects (font (size 1.27 1.27)) hide)
-    )
+    (property "Footprint" "Switch_Keyboard_Hotswap_Kailh:SW_Hotswap_Kailh_MX_plated_1.00u" (id 2) (at 127 96.52 0)
+      (effects (font (size 1.27 1.27)) hide)
+    )
